Commit message: 1.0.0.20240321124020

File: src/point_foot_robot_description/urdf/robot.urdf (robot description, URDF)
Before this commit: robot point_foot, 14 links, 13 joints
Links:
- added link contact_L, mass 1e-6
- added link contact_R, mass 1e-6
- added link world
- link abad_L: mass 1.03648983 -> 1.506; geometry visual mesh filename=package://point_foot_robot_description/meshes/abad_L_Link.S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
- link abad_R: mass 1.03648872 -> 1.506; geometry visual mesh filename=package://point_foot_robot_description/meshes/abad_R_Link.S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
- link base: mass 5.65937068 -> 7.517; geometry visual mesh filename=package://point_foot_robot_description/meshes/base_Link.STL
- link foot_L: mass 0.14047647 -> 0.153; geometry collision sphere radius=0.03; visual mesh filename=package://point_foot_robot_description/meshes/foot_L_Link.S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
- link foot_R: mass 0.14047647 -> 0.153; geometry collision sphere radius=0.03; visual mesh filename=package://point_foot_robot_description/meshes/foot_R_Link.S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
- link hip_L: mass 1.73405445 -> 2.1382; geometry visual mesh filename=package://point_foot_robot_description/meshes/hip_L_Link.STL
- link hip_R: mass 1.73405240 -> 2.1382; geometry visual mesh filename=package://point_foot_robot_description/meshes/hip_R_Link.STL
- link knee_L: mass 0.25930748 -> 0.486; geometry collision sphere radius=0.03; visual mesh filename=package://point_foot_robot_description/meshes/knee_L_Link.S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
- link knee_R: mass 0.25930895 -> 0.486; geometry collision sphere radius=0.03; visual mesh filename=package://point_foot_robot_description/meshes/knee_R_Link.S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
Joints:
- added joint contact_L_Joint: type fixed, parent foot_L, child contact_L, origin xyz=0 0 0 rpy=0 0 0, axis 0 1 0, limit lower=-0 upper=0 effort=60 velocity=50
- added joint contact_R_Joint: type revolute, parent foot_R, child contact_R, origin xyz=0 0 0 rpy=0 0 0, axis 0 1 0, limit lower=-0 upper=0 effort=60 velocity=50
- added joint fixed: type fixed, parent world, child base, origin xyz=0.0 0.0 0.1 rpy=0 0 0
- joint abad_L_joint: limit lower=-0.785398163 upper=0.383972435 effort=80.0 velocity=20.0 -> lower=-0.38397 upper=0.785398163 effort=80.0 velocity=20.0; origin xyz=0.0142 0.095 -0.08176 rpy=0 0 0 -> xyz=0.001 0.099 -0.078 rpy=0 0 0
- joint abad_R_joint: axis -1 0 0 -> 1 0 0; limit lower=-0.785398163 upper=0.383972435 effort=80.0 velocity=20.0 -> lower=-1.39626 upper=0.785398163 effort=80.0 velocity=20.0; origin xyz=0.0142 -0.095 -0.08176 rpy=0 0 0 -> xyz=0.001 -0.099 -0.078 rpy=0 0 0
- joint hip_L_joint: axis 0 -1 0 -> 0 1 0; limit lower=-1.518436449 upper=1.012290966 effort=80.0 velocity=20.0 -> lower=-1.012291 upper=1.518436 effort=80.0 velocity=20.0; origin xyz=-0.0802 0.031 0 rpy=0 0 0 -> xyz=-0.08 0.019 0.0 rpy=0 0 0
- joint hip_R_joint: limit lower=-1.518436449 upper=1.012290966 effort=80.0 velocity=20.0 -> lower=-1.518436 upper=1.012291 effort=80.0 velocity=20.0; origin xyz=-0.0802 -0.031 0 rpy=0 0 0 -> xyz=-0.08 -0.019 0.0 rpy=0 0 0
- joint knee_L_joint: limit lower=-1.396263402 upper=0.872664626 effort=80 velocity=20 -> lower=-0.872665 upper=1.396263 effort=80 velocity=20; origin xyz=-0.15 -0.031 -0.25981 rpy=0 0 0 -> xyz=-0.151 -0.019 -0.259 rpy=0 0 0
- joint knee_R_joint: limit lower=-1.396263402 upper=0.872664626 effort=80 velocity=50 -> lower=-1.396263 upper=0.872665 effort=80 velocity=50; origin xyz=-0.15 0.031 -0.25981 rpy=0 0 0 -> xyz=-0.151 0.019 -0.259 rpy=0 0 0
